Commit message: Phase 11: the arm on the base, composed rather than merged
Neither component description was modified. The arm and the base still
build and run alone, and a test asserts it -- if mounting one on the
other had needed an edit to either, this would be a third robot to
maintain instead of two that already worked. Phase 1 and Phase 10 each
spent a fixed joint on a mount frame nobody used yet; this is what they
were buying.

Two problems had to be solved for real.

BOTH COMPONENTS EMITTED THE GAZEBO SYSTEM PLUGIN. Invisible while each
robot had one subsystem, and wrong once composed: two controller
managers in one simulator process, both named controller_manager, both
loading the same controllers file. A <ros2_control> block describes
interfaces and may appear many times; the system plugin HOSTS the
manager and must appear once. They live in different files now.

EVERY MACRO READS A PROPERTY CALLED `cfg`. Fine for one robot, broken
for two: whichever config was assigned last wins and the arm gets built
from base numbers, silently, because every lookup present in both
succeeds. Rebinding `cfg` between the calls does work -- xacro expands
in document order -- and was rejected as action at a distance, the same
failure Phase 10 removed from the test harness. Each subsystem is now
wrapped in a macro that sets `cfg` inside its own body, which xacro
scopes to the invocation.

Verified running, not just parsing: four controllers active on one
manager, and `make mm-verify` drives and manipulates CONCURRENTLY --
the base travelled 0.345 m while the arm moved 0.396 rad, with the
trajectory goal accepted mid-drive. Run sequentially, two controllers
that quietly share a resource still look fine.

There is no mm_controllers.yaml. The launch merges the two subsystems'
configs and prefixes the arm's joint names, because a committed third
file would hold the same joint list twice and adding an arm joint would
leave the composed robot driving the old set. The merge refuses a
disagreement rather than resolving it: both configs set
controller_manager.update_rate, and letting one win silently would run
the robot at a rate neither file states.

Can it tip itself over? The arm is a large fraction of the mass and it
moves, so that is a question about the whole workspace, not one pose.
A sweep of the joint limits carrying the payload, checked against all
four wheel contacts, no simulator involved:

  threevn_mm_v1             1.267 kg  reach +0.244 m  +38.8 mm (rear)
  threevn_mm_v1_long_reach  1.313 kg  reach +0.338 m  +30.0 mm (rear)

against a required 21.0 mm. The measurement corrected the intuition
this was built on: the binding edge is the REAR, not the front. The
support rectangle is narrower front-to-back, so reaching forward looks
like the danger, and mounting the arm behind centre does buy margin
against it -- while spending that margin at the rear. The profile
comment claiming it was free is now the measured trade.

Also fixed: the base's root joint was still called chassis_joint, left
over from Phase 10 renaming the link it points at.

Every mass here is provenance: estimated. These margins are arithmetic
on guesses and must be re-run once anything is weighed.

Nav2 is NOT in this phase and the roadmap now says so.

Co-Authored-By: Claude Opus 5 <noreply@anthropic.com>

File: src/threevn_robot_description/urdf/base/base.ros2_control.xacro (robot description, xacro)
@@ -52,13 +52,4 @@
     </ros2_control>
     <xacro:if value="${'$(arg target)' == 'gz'}">
-      <gazebo>
-        <plugin filename="gz_ros2_control-system"
-                name="gz_ros2_control::GazeboSimROS2ControlPlugin">
-          <xacro:if value="${'$(arg controllers_file)' != ''}">
-            <parameters>$(arg controllers_file)</parameters>
-          </xacro:if>
-          <controller_manager_name>controller_manager</controller_manager_name>
-        </plugin>
-      </gazebo>
       <!-- Skid steer scrubs. Without tuned friction Gazebo either grips
            so hard the chassis will not rotate, or slides like ice. These

File: src/threevn_robot_description/urdf/base/base_macro.xacro (robot description, xacro)
@@ -57,5 +57,8 @@
   <xacro:macro name="threevn_base" params="parent prefix">
     <xacro:property name="chassis" value="${cfg['links']['base_link']}"/>
-    <joint name="${prefix}chassis_joint" type="fixed">
+    <!-- base_footprint -> base_link. Named base_joint to match what
+         it connects; it was chassis_joint until the link it points at
+         stopped being chassis_link. -->
+    <joint name="${prefix}base_joint" type="fixed">
       <parent link="${parent}"/>
       <child link="${prefix}base_link"/>

File: src/threevn_robot_description/urdf/ros2_control/arm.ros2_control.xacro (robot description, xacro)
@@ -91,35 +91,4 @@
       <xacro:threevn_joint_ifaces name="gripper_left_finger_joint" prefix="${prefix}"/>
     </ros2_control>
-    <!--
-      Gazebo needs a system plugin to host controller_manager inside the
-      simulator process. Emitted ONLY for target=gz, so a real-robot or
-      mock build never references a Gazebo library at all.
-      test_ros2_control_targets.py asserts exactly that, and that
-      assertion IS the architecture.
-    -->
-    <xacro:if value="${'$(arg target)' == 'gz'}">
-      <gazebo>
-        <plugin filename="gz_ros2_control-system"
-                name="gz_ros2_control::GazeboSimROS2ControlPlugin">
-          <!--
-            The controllers file is PASSED IN, not looked up.
-            It used to be $(find threevn_bringup)/config/controllers.yaml,
-            which inverted the dependency direction: threevn_bringup
-            depends on this package, so this package must not reach back
-            into it. That went unnoticed because a fully sourced
-            workspace resolves the path anyway - it only surfaced when CI
-            built and tested this package in isolation and xacro raised
-            PackageNotFoundError.
-            threevn_sim depends on both and supplies the path, so the
-            dependency graph stays acyclic and the description stays
-            standalone.
-          -->
-          <xacro:if value="${'$(arg controllers_file)' != ''}">
-            <parameters>$(arg controllers_file)</parameters>
-          </xacro:if>
-          <controller_manager_name>controller_manager</controller_manager_name>
-        </plugin>
-      </gazebo>
-    </xacro:if>
   </xacro:macro>
 </robot>

File: src/threevn_robot_description/urdf/threevn_arm.urdf.xacro (robot description, xacro)
@@ -42,4 +42,5 @@
   <xacro:include filename="$(find threevn_robot_description)/urdf/ros2_control/arm.ros2_control.xacro"/>
   <xacro:include filename="$(find threevn_robot_description)/urdf/gazebo/materials.gazebo.xacro"/>
+  <xacro:include filename="$(find threevn_robot_description)/urdf/ros2_control/gz_control_plugin.xacro"/>
   <!-- The kinematic root. Zero inertia, pure reference frame: it is the
        projection of the robot onto the floor, and in Phase 11 it becomes
@@ -58,3 +59,8 @@
     <xacro:threevn_gazebo_materials prefix="${prefix}"/>
   </xacro:if>
+  <!-- Exactly one controller_manager, however many ros2_control blocks
+       the robot has. See gz_control_plugin.xacro. -->
+  <xacro:if value="${'$(arg target)' == 'gz'}">
+    <xacro:threevn_gz_control_plugin/>
+  </xacro:if>
 </robot>

File: src/threevn_robot_description/urdf/threevn_base.urdf.xacro (robot description, xacro)
@@ -19,4 +19,5 @@
   <xacro:include filename="$(find threevn_robot_description)/urdf/base/base_macro.xacro"/>
   <xacro:include filename="$(find threevn_robot_description)/urdf/base/base.ros2_control.xacro"/>
+  <xacro:include filename="$(find threevn_robot_description)/urdf/ros2_control/gz_control_plugin.xacro"/>
   <!-- Same root name as the arm. It is the robot's projection onto the
        floor either way, which is what lets Phase 11 join them without
@@ -25,3 +26,8 @@
   <xacro:threevn_base parent="${prefix}base_footprint" prefix="${prefix}"/>
   <xacro:threevn_base_ros2_control prefix="${prefix}"/>
+  <!-- Exactly one controller_manager, however many ros2_control blocks
+       the robot has. See gz_control_plugin.xacro. -->
+  <xacro:if value="${'$(arg target)' == 'gz'}">
+    <xacro:threevn_gz_control_plugin/>
+  </xacro:if>
 </robot>
